File: hardware/eagle/main_SMD_FET.brd (EAGLE design)
At the start: 40 x 31.7 mm, 44 parts, among them IC1 R-78E3.3-1.0, IC2 INA186A1QDCKRQ1, IC3 ESP-12E/F, J4 1727078, Q1 IRFU3710ZPBF, Q2 IRFU3710ZPBF, Q3 IRFU3710ZPBF, Q4 IRFU3710ZPBF

Commit message: initial
Parts:
- Q1, Q2, Q3, Q4: value IRFU3710ZPBF -> IPD031N06; device SamacSys_Parts:TO229P239X654X978-3P -> SamacSys_Parts:IPD031N06L3GATMA1
- moved C6 8.98 mm to (19.1, 16.8)
- moved C10 8.53 mm to (18.7, 25.4)
- moved C11 7.03 mm to (19.4, 21.9), flipped to the top, turned to 0 degrees
- moved C9 6.24 mm to (18.7, 13.3), flipped to the top, turned to 0 degrees
- moved R15 6.07 mm to (19.7, 14.9), turned to 90 degrees
- moved R17 5.62 mm to (19.4, 23.5), turned to 90 degrees
- moved Q4 5.55 mm to (11.1, 13.0), flipped to the bottom, turned to 270 degrees
- moved R9 5.41 mm to (26.4, 9.84), turned to 90 degrees
- moved Q2 5.28 mm to (11.1, 21.6), flipped to the bottom, turned to 270 degrees
- moved R18 4.49 mm to (20.0, 23.5), flipped to the top, turned to 270 degrees
- moved R16 3.81 mm to (19.4, 14.9), flipped to the top, turned to 270 degrees
- moved Q1 2.93 mm to (11.1, 22.2), turned to 90 degrees
- moved IC3 2.88 mm to (30.5, 17.8)
- moved R10 2.88 mm to (27.9, 13.7)
- moved R8 2.88 mm to (38.1, 22.2)
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Routing:
- net N$7: track 21.8 -> 37.3 mm, vias 0 -> 3
- net W: track 11.8 -> 18.8 mm
- net G: track 12.5 -> 19.3 mm
- net N$3: track 9.49 -> 14.1 mm, vias 0 -> 1
- net N$13: track 31.6 -> 27.4 mm
- net N$1: track 38.4 -> 42.0 mm
- net W_PIN: track 20.1 -> 16.6 mm
- net R_PIN: track 13.0 -> 9.62 mm, vias 1 -> 0
- net IN_1_PIN: track 18.6 -> 21.3 mm
- net IN_2_PIN: track 20.8 -> 23.4 mm
- net B: track 12.2 -> 14.8 mm
- net N$10: track 0.00 -> 2.53 mm, vias 0 -> 1
- net B_PIN: track 6.63 -> 4.22 mm, vias 1 -> 0
- net G_PIN: track 5.13 -> 7.11 mm
- net R: track 13.3 -> 15.3 mm
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
Commit message: Konturanpassung
Parts:
- removed IC2: INA186A1QDCKRQ1, SamacSys_Parts:SOP65P210X110-6N
- removed R13, R14: (no value), rcl:R0402
- added C12: 100n, rcl:C0603
- added IC4: INA301A1IDGKR, SamacSys_Parts:SOP65P490X110-8N
- moved C5 3.88 mm to (11.4, 6.67), turned to 0 degrees
- moved L1 2.25 mm to (11.4, 2.86)
- moved C10 0.64 mm to (18.7, 26.0)
- moved Q2 0.64 mm to (11.1, 22.2)
- moved R5 0.64 mm to (9.21, 27.9)
- moved IC1 0.63 mm to (19.1, 2.22)
- moved R17 0.63 mm to (19.4, 24.1)
- moved R7 0.32 mm to (34.0, 21.9)
- moved R8 0.32 mm to (38.1, 21.9)
- moved R10 0.32 mm to (27.9, 14.0)
- moved R11 0.32 mm to (29.8, 14.0)
- moved D1 0.32 mm to (12.4, 28.6)
- moved D2 0.32 mm to (12.4, 28.6)
- moved R3 0.32 mm to (19.4, 21.9)
Connections:
- removed net N$8: IC2.1, R13.1, R14.1
- net +3V3: now also C12.2, IC4.1; no longer IC2.3, R13.2
- net GND: now also C12.1, IC4.4, IC4.7; no longer IC2.2, IC2.5, R14.2
- net N$1: now also IC4.2; no longer IC2.6
- net N$7: now also IC4.8; no longer IC2.4
Routing:
- net GND: track 36.6 -> 11.3 mm, vias 0 -> 12
- net +3V3: track 59.9 -> 56.1 mm
- net N$1: track 42.0 -> 38.5 mm
- net N$8: track 3.01 -> 0.00 mm
- net W_PIN: track 16.6 -> 18.4 mm
- net N$9: track 7.49 -> 9.21 mm
- net G: track 19.3 -> 17.7 mm
- net N$13: track 27.4 -> 28.4 mm
- net W: track 18.8 -> 17.9 mm
- net N$7: track 37.3 -> 38.1 mm, vias 3 -> 6
- net N$25: track 3.69 -> 4.32 mm
- net IN_1_PIN: track 21.3 -> 21.8 mm
Other:
- board size 40 x 31.7 mm -> 40 x 31.8 mm
