File: hardware/eagle/main_SMD_FET.sch (EAGLE design)
At the start: 43 parts, among them IC1 R-78E3.3-1.0, IC3 ESP-12E/F, IC4 INA301A1IDGKR, J4 1727078, Q1 IPD031N06, Q2 IPD031N06, Q3 IPD031N06, Q4 IPD031N06

Commit message: tiefpass eingefügt. Leiterbahn etwas breiter für DC/DC wandler
Parts:
- added C13: 100n, rcl:C-EUC0603
- added R13: 10k, rcl:R-EU_R0402
- C3, C4: value (none) -> 4µ7
- C5: value (none) -> 1µ
- R12: value PCS1206DR0100ET -> 0R005
Connections:
- removed net N$1: IC3.ADC, IC4.OUT
- new net N$: C13.2, IC3.ADC, R13.2
- new net N$8: IC4.OUT, R13.1
- net GND: now also C13.1
Changed lines of the file:
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@@
 <part name="+3V1" library="supply1" library_urn="urn:adsk.eagle:library:371" deviceset="+3V3" device=""/>
 <part name="P+1" library="supply1" library_urn="urn:adsk.eagle:library:371" deviceset="V+" device=""/>
-<part name="R12" library="SamacSys_Parts" deviceset="PCS1206DR0100ET" device="" override_package3d_urn="urn:adsk.eagle:package:27074030/2" override_package_urn="urn:adsk.eagle:footprint:27074031/1"/>
+<part name="R12" library="SamacSys_Parts" deviceset="PCS1206DR0100ET" device="" override_package3d_urn="urn:adsk.eagle:package:27074030/2" override_package_urn="urn:adsk.eagle:footprint:27074031/1" value="0R005"/>
 <part name="P+2" library="supply1" library_urn="urn:adsk.eagle:library:371" deviceset="V+" device=""/>
 <part name="GND21" library="supply1" library_urn="urn:adsk.eagle:library:371" deviceset="GND" device=""/>
@@
 <part name="GND23" library="supply1" library_urn="urn:adsk.eagle:library:371" deviceset="GND" device=""/>
 <part name="L1" library="SamacSys_Parts" deviceset="RLS-126-R" device="" override_package3d_urn="urn:adsk.eagle:package:27099534/2" override_package_urn="urn:adsk.eagle:footprint:27099535/1"/>
-<part name="C3" library="rcl" library_urn="urn:adsk.eagle:library:334" deviceset="C-EU" device="C0603" package3d_urn="urn:adsk.eagle:package:23616/2"/>
-<part name="C4" library="rcl" library_urn="urn:adsk.eagle:library:334" deviceset="C-EU" device="C1206" package3d_urn="urn:adsk.eagle:package:23618/2"/>
-<part name="C5" library="rcl" library_urn="urn:adsk.eagle:library:334" deviceset="C-EU" device="C1206" package3d_urn="urn:adsk.eagle:package:23618/2"/>
+<part name="C3" library="rcl" library_urn="urn:adsk.eagle:library:334" deviceset="C-EU" device="C0603" package3d_urn="urn:adsk.eagle:package:23616/2" value="4µ7"/>
+<part name="C4" library="rcl" library_urn="urn:adsk.eagle:library:334" deviceset="C-EU" device="C1206" package3d_urn="urn:adsk.eagle:package:23618/2" value="4µ7"/>
+<part name="C5" library="rcl" library_urn="urn:adsk.eagle:library:334" deviceset="C-EU" device="C1206" package3d_urn="urn:adsk.eagle:package:23618/2" value="1µ"/>
 <part name="IC1" library="SamacSys_Parts" deviceset="R-78E3.3-1.0" device="" override_package3d_urn="urn:adsk.eagle:package:26628885/2" override_package_urn="urn:adsk.eagle:footprint:26628886/1"/>
 <part name="IC3" library="esp-12e-f" deviceset="ESP-12E/F" device="" override_package3d_urn="urn:adsk.eagle:package:27056995/2" override_package_urn="urn:adsk.eagle:footprint:27056996/1"/>
@@
 <part name="C12" library="rcl" library_urn="urn:adsk.eagle:library:334" deviceset="C-EU" device="C0603" package3d_urn="urn:adsk.eagle:package:23616/2" value="100n"/>
 <part name="GND19" library="supply1" library_urn="urn:adsk.eagle:library:371" deviceset="GND" device=""/>
-<part name="+3V2" library="supply1" library_urn="urn:adsk.eagle:library:371" deviceset="+3V3" device=""/>
+<part name="R13" library="rcl" library_urn="urn:adsk.eagle:library:334" deviceset="R-EU_" device="R0402" package3d_urn="urn:adsk.eagle:package:23547/3" value="10k"/>
+<part name="C13" library="rcl" library_urn="urn:adsk.eagle:library:334" deviceset="C-EU" device="C0603" package3d_urn="urn:adsk.eagle:package:23616/2" value="100n"/>
+<part name="GND20" library="supply1" library_urn="urn:adsk.eagle:library:371" deviceset="GND" device=""/>
 </parts>
 <sheets>
@@
 <attribute name="VALUE" x="157.48" y="205.74" size="1.778" layer="96"/>
 </instance>
-<instance part="+3V2" gate="G$1" x="160.02" y="238.76" smashed="yes">
-<attribute name="VALUE" x="157.48" y="233.68" size="1.778" layer="96" rot="R90"/>
+<instance part="R13" gate="G$1" x="170.18" y="223.52" smashed="yes">
+<attribute name="NAME" x="166.37" y="225.0186" size="1.778" layer="95"/>
+<attribute name="VALUE" x="166.37" y="220.218" size="1.778" layer="96"/>
+</instance>
+<instance part="C13" gate="G$1" x="180.34" y="215.9" smashed="yes" rot="R180">
+<attribute name="NAME" x="178.816" y="215.519" size="1.778" layer="95" rot="R180"/>
+<attribute name="VALUE" x="178.816" y="220.599" size="1.778" layer="96" rot="R180"/>
+</instance>
+<instance part="GND20" gate="1" x="180.34" y="208.28" smashed="yes">
+<attribute name="VALUE" x="177.8" y="205.74" size="1.778" layer="96"/>
 </instance>
 </instances>
@@
 <wire x1="149.86" y1="236.22" x2="149.86" y2="226.06" width="0.1524" layer="91"/>
 <wire x1="149.86" y1="226.06" x2="147.32" y2="226.06" width="0.1524" layer="91"/>
-</segment>
-<segment>
 <pinref part="C12" gate="G$1" pin="2"/>
-<pinref part="+3V2" gate="G$1" pin="+3V3"/>
-<wire x1="160.02" y1="236.22" x2="160.02" y2="220.98" width="0.1524" layer="91"/>
+<wire x1="160.02" y1="226.06" x2="160.02" y2="220.98" width="0.1524" layer="91"/>
+<wire x1="149.86" y1="226.06" x2="160.02" y2="226.06" width="0.1524" layer="91"/>
+<junction x="149.86" y="226.06"/>
 </segment>
 </net>
@@
 <pinref part="GND19" gate="1" pin="GND"/>
 <wire x1="160.02" y1="210.82" x2="160.02" y2="213.36" width="0.1524" layer="91"/>
+</segment>
+<segment>
+<pinref part="GND20" gate="1" pin="GND"/>
+<pinref part="C13" gate="G$1" pin="1"/>
+<wire x1="180.34" y1="210.82" x2="180.34" y2="213.36" width="0.1524" layer="91"/>
 </segment>
 </net>
@@
 </segment>
 </net>
-<net name="N$1" class="0">
+<net name="N$" class="0">
 <segment>
 <wire x1="208.28" y1="223.52" x2="208.28" y2="190.5" width="0.1524" layer="91"/>
 <wire x1="208.28" y1="190.5" x2="238.76" y2="190.5" width="0.1524" layer="91"/>
 <pinref part="IC3" gate="G$1" pin="ADC"/>
-<pinref part="IC4" gate="G$1" pin="OUT"/>
-<wire x1="147.32" y1="223.52" x2="208.28" y2="223.52" width="0.1524" layer="91"/>
+<wire x1="175.26" y1="223.52" x2="180.34" y2="223.52" width="0.1524" layer="91"/>
+<pinref part="R13" gate="G$1" pin="2"/>
+<pinref part="C13" gate="G$1" pin="2"/>
+<wire x1="180.34" y1="223.52" x2="208.28" y2="223.52" width="0.1524" layer="91"/>
+<wire x1="180.34" y1="220.98" x2="180.34" y2="223.52" width="0.1524" layer="91"/>
+<junction x="180.34" y="223.52"/>
 </segment>
 </net>
@@
 </segment>
 </net>
+<net name="N$8" class="0">
+<segment>
+<pinref part="IC4" gate="G$1" pin="OUT"/>
+<wire x1="147.32" y1="223.52" x2="165.1" y2="223.52" width="0.1524" layer="91"/>
+<pinref part="R13" gate="G$1" pin="1"/>
+</segment>
+</net>

Commit message: dokumentation
Parts:
- D1, D2: value BZX84CSMD -> BZX84C3V3
Changed lines of the file:
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@@
 <part name="J4" library="SamacSys_Parts_PHOENIX" deviceset="1727078" device="" override_package3d_urn="urn:adsk.eagle:package:26529790/2" override_package_urn="urn:adsk.eagle:footprint:15226074/1"/>
 <part name="GND6" library="supply1" library_urn="urn:adsk.eagle:library:371" deviceset="GND" device=""/>
-<part name="D1" library="diode" library_urn="urn:adsk.eagle:library:210" deviceset="BZX84CSMD" device="" package3d_urn="urn:adsk.eagle:package:43403/2"/>
-<part name="D2" library="diode" library_urn="urn:adsk.eagle:library:210" deviceset="BZX84CSMD" device="" package3d_urn="urn:adsk.eagle:package:43403/2"/>
+<part name="D1" library="diode" library_urn="urn:adsk.eagle:library:210" deviceset="BZX84CSMD" device="" package3d_urn="urn:adsk.eagle:package:43403/2" value="BZX84C3V3"/>
+<part name="D2" library="diode" library_urn="urn:adsk.eagle:library:210" deviceset="BZX84CSMD" device="" package3d_urn="urn:adsk.eagle:package:43403/2" value="BZX84C3V3"/>
 <part name="R5" library="rcl" library_urn="urn:adsk.eagle:library:334" deviceset="R-EU_" device="R0603" package3d_urn="urn:adsk.eagle:package:23555/3" value="10k"/>
 <part name="R6" library="rcl" library_urn="urn:adsk.eagle:library:334" deviceset="R-EU_" device="R0603" package3d_urn="urn:adsk.eagle:package:23555/3" value="10k"/>
@@
 <part name="GND22" library="supply1" library_urn="urn:adsk.eagle:library:371" deviceset="GND" device=""/>
 <part name="GND23" library="supply1" library_urn="urn:adsk.eagle:library:371" deviceset="GND" device=""/>
-<part name="L1" library="SamacSys_Parts" deviceset="RLS-126-R" device="" override_package3d_urn="urn:adsk.eagle:package:27099534/2" override_package_urn="urn:adsk.eagle:footprint:27099535/1"/>
+<part name="L1" library="SamacSys_Parts" deviceset="RLS-126-R" device="" override_package3d_urn="urn:adsk.eagle:package:27099534/2" override_package_urn="urn:adsk.eagle:footprint:27099535/1" override_locally_modified="yes"/>
 <part name="C3" library="rcl" library_urn="urn:adsk.eagle:library:334" deviceset="C-EU" device="C0603" package3d_urn="urn:adsk.eagle:package:23616/2" value="4µ7"/>
 <part name="C4" library="rcl" library_urn="urn:adsk.eagle:library:334" deviceset="C-EU" device="C1206" package3d_urn="urn:adsk.eagle:package:23618/2" value="4µ7"/>
 <part name="C5" library="rcl" library_urn="urn:adsk.eagle:library:334" deviceset="C-EU" device="C1206" package3d_urn="urn:adsk.eagle:package:23618/2" value="1µ"/>
-<part name="IC1" library="SamacSys_Parts" deviceset="R-78E3.3-1.0" device="" override_package3d_urn="urn:adsk.eagle:package:26628885/2" override_package_urn="urn:adsk.eagle:footprint:26628886/1"/>
+<part name="IC1" library="SamacSys_Parts" deviceset="R-78E3.3-1.0" device="" override_package3d_urn="urn:adsk.eagle:package:26628885/2" override_package_urn="urn:adsk.eagle:footprint:26628886/1" override_locally_modified="yes"/>
 <part name="IC3" library="esp-12e-f" deviceset="ESP-12E/F" device="" override_package3d_urn="urn:adsk.eagle:package:27056995/2" override_package_urn="urn:adsk.eagle:footprint:27056996/1"/>
 <part name="PROG" library="Tyco_By_element14_Batch_1" deviceset="PINHD-2X2" device="" override_package3d_urn="urn:adsk.eagle:package:27057090/2" override_package_urn="urn:adsk.eagle:footprint:27057102/1"/>
@@
 <part name="C10" library="rcl" library_urn="urn:adsk.eagle:library:334" deviceset="C-EU" device="C0402" package3d_urn="urn:adsk.eagle:package:23626/2"/>
 <part name="C11" library="rcl" library_urn="urn:adsk.eagle:library:334" deviceset="C-EU" device="C0402" package3d_urn="urn:adsk.eagle:package:23626/2"/>
-<part name="Q1" library="SamacSys_Parts" deviceset="IPD031N06L3GATMA1" device="" override_package3d_urn="urn:adsk.eagle:package:27099134/2" override_package_urn="urn:adsk.eagle:footprint:27099162/1" value="IPD031N06"/>
+<part name="Q1" library="SamacSys_Parts" deviceset="IPD031N06L3GATMA1" device="" override_package3d_urn="urn:adsk.eagle:package:27099134/2" override_package_urn="urn:adsk.eagle:footprint:27099162/1" override_locally_modified="yes" value="IPD031N06"/>
 <part name="GND17" library="supply1" library_urn="urn:adsk.eagle:library:371" deviceset="GND" device=""/>
-<part name="Q2" library="SamacSys_Parts" deviceset="IPD031N06L3GATMA1" device="" override_package3d_urn="urn:adsk.eagle:package:27098765/2" override_package_urn="urn:adsk.eagle:footprint:27098804/1" value="IPD031N06"/>
-<part name="Q3" library="SamacSys_Parts" deviceset="IPD031N06L3GATMA1" device="" override_package3d_urn="urn:adsk.eagle:package:27098577/2" override_package_urn="urn:adsk.eagle:footprint:27098578/1" value="IPD031N06"/>
-<part name="Q4" library="SamacSys_Parts" deviceset="IPD031N06L3GATMA1" device="" override_package3d_urn="urn:adsk.eagle:package:27056889/3" override_package_urn="urn:adsk.eagle:footprint:27056890/1" value="IPD031N06"/>
+<part name="Q2" library="SamacSys_Parts" deviceset="IPD031N06L3GATMA1" device="" override_package3d_urn="urn:adsk.eagle:package:27098765/2" override_package_urn="urn:adsk.eagle:footprint:27098804/1" override_locally_modified="yes" value="IPD031N06"/>
+<part name="Q3" library="SamacSys_Parts" deviceset="IPD031N06L3GATMA1" device="" override_package3d_urn="urn:adsk.eagle:package:27098577/2" override_package_urn="urn:adsk.eagle:footprint:27098578/1" override_locally_modified="yes" value="IPD031N06"/>
+<part name="Q4" library="SamacSys_Parts" deviceset="IPD031N06L3GATMA1" device="" override_package3d_urn="urn:adsk.eagle:package:27056889/3" override_package_urn="urn:adsk.eagle:footprint:27056890/1" override_locally_modified="yes" value="IPD031N06"/>
 <part name="IC4" library="SamacSys_Parts" deviceset="INA301A1IDGKR" device="" override_package3d_urn="urn:adsk.eagle:package:27074000/2" override_package_urn="urn:adsk.eagle:footprint:27074001/1"/>
 <part name="GND24" library="supply1" library_urn="urn:adsk.eagle:library:371" deviceset="GND" device=""/>
@@
 </instance>
 <instance part="J4" gate="G$1" x="27.94" y="198.12" smashed="yes" rot="MR0">
-<attribute name="NAME" x="11.43" y="205.74" size="1.778" layer="95" rot="MR0" align="center-left"/>
-<attribute name="VALUE" x="11.43" y="203.2" size="1.778" layer="96" rot="MR0" align="center-left"/>
+<attribute name="NAME" x="13.97" y="205.74" size="1.778" layer="95" rot="MR180" align="center-left"/>
+<attribute name="VALUE" x="13.97" y="203.2" size="1.778" layer="96" rot="MR180" align="center-left"/>
 </instance>
 <instance part="GND6" gate="1" x="30.48" y="170.18" smashed="yes">
@@
 <segment>
 <wire x1="312.42" y1="187.96" x2="276.86" y2="187.96" width="0.1524" layer="91"/>
-<label x="281.94" y="187.96" size="1.778" layer="95"/>
+<label x="304.8" y="187.96" size="1.778" layer="95"/>
 <pinref part="IC3" gate="G$1" pin="IO5"/>
 </segment>
